Commit message: add motion planning examples

File: ar1440_description/urdf/ar1440_macro.xacro (robot description, xacro)
@@ -183,5 +183,5 @@
     <link name="${prefix}world" />
     <joint name="${prefix}base_link-base" type="fixed">
-        <origin xyz="0 0 0.450" rpy="0 0 0"/>
+        <origin xyz="0 0 0.0" rpy="0 0 0"/>
         <child link="${prefix}base_link"/>
         <parent link="${prefix}world"/>
